Commit message: relative paths

File: bluerov2_ignition/urdf/bluerov2.urdf (robot description, URDF)
Before this commit: robot bluerov2, 11 links, 10 joints
Links:
- link bluerov2/base_link: geometry collision box size=0.464714527531344 0.29044657970709 0.116178631882836; visual mesh filename=file://$(find bluerov2_description)/meshes/bluerov2_noprop.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
- link bluerov2/thruster1: geometry visual mesh filename=file://$(find bluerov2_description)/meshes/bluerov2_propcw.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
- link bluerov2/thruster2: geometry visual mesh filename=file://$(find bluerov2_description)/meshes/bluerov2_propcw.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
- link bluerov2/thruster3: geometry visual mesh filename=file://$(find bluerov2_description)/meshes/bluerov2_propcw.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
- link bluerov2/thruster4: geometry visual mesh filename=file://$(find bluerov2_description)/meshes/bluerov2_propcw.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
- link bluerov2/thruster5: geometry visual mesh filename=file://$(find bluerov2_description)/meshes/bluerov2_propcw.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
- link bluerov2/thruster6: geometry visual mesh filename=file://$(find bluerov2_description)/meshes/bluerov2_propcw.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
