Commit message: compat with auv_control

File: bluerov2_description/urdf/bluerov2.xacro (robot description, xacro)
@@ -4,22 +4,18 @@
   <!-- thruster joints are fixed if not for gazebo use -->
   <xacro:arg name="simulation" default="true"/>
+  <xacro:arg name="camera" default="true"/>
   <xacro:arg name="density" default="1000"/>
   <xacro:property name="ns" value="$(arg namespace)"/>
   <xacro:property name="density" value="$(arg density)"/>
   <!-- Main body -->
-  <xacro:property name="mass" value="10"/>
   <xacro:property name="x_size" value="0.40"/>
   <xacro:property name="y_size" value="0.25"/>
   <xacro:property name="z_size" value="0.1"/>
-<!-- <xacro:property name="mass" value="147.8671"/> -->
-  <!--<xacro:property name="x_size" value="2."/>
-  <xacro:property name="y_size" value="0.3"/>
-  <xacro:property name="z_size" value="0.246445166667"/> -->
+    <xacro:property name="mass" value="14.8"/>
   <!-- other props -->
   <xacro:property name="prop_mass" value="0.07"/>
   <xacro:property name="PI" value="3.1415927"/>
-  <!-- to set correct buoyancy volume -->
-  <xacro:property name="total_mass" value="${mass + 0*prop_mass}"/>
-  <xacro:property name="buoyant_correction" value="${pow(1.05*total_mass/(density*x_size*y_size*z_size), 1./3)}"/>
+  <!-- to set correct buoyancy volume with 1 % positive factor -->
+  <xacro:property name="buoyant_correction" value="${pow(1.01*(mass + 6*prop_mass)/(density*x_size*y_size*z_size), 1./3)}"/>
   <!-- Center of gravity -->
   <xacro:property name="z_cog" value="${-buoyant_correction*z_size}"/>
@@ -29,38 +25,43 @@
     <link name="${ns}/base_link">
     <inertial>
-        <mass value="${mass}" />
+        <mass value="${mass}"/>
         <origin xyz="0 0 ${z_cog}"/>
-        <!-- <inertia ixx="525.39" ixy="1.44" ixz="33.41" iyy="794.20" iyz="2.6" izz="691.23"/> -->
-        <inertia
+    <!-- BlueROV2 values from "Model Predictive Control for the BlueROV2",
+        Emil Már Einarsson, Andris Lipenitis, Master thesis, 2020
+        for now make Ignition crash?-->
+<!--         <inertia ixx="0.21" ixy="0.00" ixz="0.00" iyy="0.245" iyz="0.00" izz="0.245"/> -->
+        <inertia ixx="5.2539" ixy="0.0144" ixz="0.3341" iyy="7.9420" iyz="0.026" izz="6.9123"/>
+            <!-- Perfect rectangle -->
+<!--        <inertia
         ixx="${mass/12*(y_size*y_size+z_size*z_size)}" ixy="0.0" ixz="0.0"
         iyy="${mass/12*(x_size*x_size + z_size*z_size)}" iyz="0.0"
-        izz="${mass/12*(x_size*x_size + y_size*y_size)}" />
-<!--        <inertia
-        ixx="3.0" ixy="0.0" ixz="0.0"
-        iyy="4.98" iyz="0.0"
-        izz="4.98" />-->
+        izz="${mass/12*(x_size*x_size + y_size*y_size)}" />-->
     </inertial>
     <visual>
         <geometry>
-        <mesh filename="${visual_mesh_file}" scale="1 1 1" />
+        <mesh filename="${visual_mesh_file}"/>
         </geometry>
     </visual>
     <collision>
-<!--        <geometry>
-            <mesh filename="${collision_mesh_file}" scale="1 1 1" />
-        </geometry>-->
+        <!-- Box adjusted for buoyancy -->
         <geometry>
             <box size="${x_size*buoyant_correction} ${y_size*buoyant_correction} ${z_size*buoyant_correction}"/>
-<!--             <box size="2 0.3 0.246445166667"/>             -->
         </geometry>
     </collision>
     </link>
-<!--   <xacro:include filename="hydrodynamics.xacro"/> -->
-  <xacro:include filename="thrusters.xacro" />
-<!--   <xacro:include filename="sensors.xacro"/> -->
+<xacro:include filename="hydrodynamics.xacro"/>
+<xacro:include filename="thrusters.xacro"/>
+  <xacro:include filename="sensors.xacro"/>
 <!-- other Gazebo plugins -->
 <xacro:if value="$(arg simulation)">
     <gazebo>
         <plugin filename="libignition-gazebo-joint-state-publisher-system.so" name="ignition::gazebo::systems::JointStatePublisher"/>
+        <plugin
+            filename="libignition-gazebo-odometry-publisher-system.so"
+            name="ignition::gazebo::systems::OdometryPublisher">
+            <odom_frame>${ns}/odom</odom_frame>
+            <robot_base_frame>${ns}/base_link</robot_base_frame>
+            <odom_publish_frequency>10</odom_publish_frequency>
+        </plugin>
         <plugin
             filename="libignition-gazebo-pose-publisher-system.so"

File: bluerov2_description/urdf/hydrodynamics.xacro (robot description, xacro)
@@ -7,48 +7,45 @@
     <!-- Ignition notations from Handbook of Marine Craft, Fossen, 2011 -->
     <link_name>${ns}/base_link</link_name>
-<!-- Thetys -->
-        <xDotU>-4.876161</xDotU>
-        <yDotV>-126.324739</yDotV>
-        <zDotW>-126.324739</zDotW>
-        <kDotP>0</kDotP>
-        <mDotQ>-33.46</mDotQ>
-        <nDotR>-33.46</nDotR>
-        <xUU>-6.2282</xUU>
-        <xU>0</xU>
-        <yVV>-601.27</yVV>
-        <yV>0</yV>
-        <zWW>-601.27</zWW>
-        <zW>0</zW>
-        <kPP>-0.1916</kPP>
-        <kP>0</kP>
-        <mQQ>-632.698957</mQQ>
-        <mQ>0</mQ>
-        <nRR>-632.698957</nRR>
-        <nR>0</nR>
     <!-- BlueROV2 heavy values from "6-DoF Modelling and Control of a Remotely Operated Vehicle"
         Wu, Master thesis, Flinder University, 2018  -->
     <!-- Negative diagonal values of added mass matrix [Fossen (6.38)] -->
-<!--    <xDotU>5.5</xDotU>
-    <yDotV>12.7</yDotV>
-    <zDotW>14.57</zDotW>
-    <kDotP>0.12</kDotP>
-    <mDotQ>0.12</mDotQ>
-    <nDotR>0.12</nDotR>-->
-    <!-- BlueROV2 values from "Numerical Modelling and Experimental Testing of the Hydrodynamic Characteristics
+    <xDotU>-5.5</xDotU>
+    <yDotV>-12.7</yDotV>
+    <zDotW>-14.57</zDotW>
+    <kDotP>-0.12</kDotP>
+    <mDotQ>-0.12</mDotQ>
+    <nDotR>-0.12</nDotR>
+    <!-- From "Numerical Modelling and Experimental Testing of the Hydrodynamic Characteristics
         for an Open-Frame Remotely Operated Vehicle",  Li et al, Marine Science and Engineering, 2020         -->
     <!-- Negative linear damping [Fossen (6.62)] -->
-<!--    <xU>1.31</xU>
-    <yV>9.14</yV>
-    <zW>2.015</zW>
-    <kP>0.</kP>
-    <mQ>0.</mQ>
-    <nR>0.</nR>-->
+<!--    <xU>-1.31</xU>
+    <yV>-9.14</yV>
+    <zW>-2.015</zW>
+    <kP>-0.</kP>
+    <mQ>-0.</mQ>
+    <nR>-0.</nR>-->
     <!-- Negative quadratic damping [Fossen (6.62)] -->
 <!--    <xUU>38.169</xUU>
-    <yVV>129.66</yVV>
-    <zWW>243.25</zWW>
-    <kPP>4.86</kPP>
-    <mQQ>4.86</mQQ>
-    <nRR>4.86</nRR>-->
+    <yVV>-129.66</yVV>
+    <zWW>-243.25</zWW>
+    <kPP>-4.86</kPP>
+    <mQQ>-4.86</mQQ>
+    <nRR>-4.86</nRR>-->
+    <!-- BlueROV2 values from "Model Predictive Control for the BlueROV2",
+        Emil Már Einarsson, Andris Lipenitis, Master thesis, 2020  -->
+    <!-- Negative linear damping -->
+    <xU>-25.15</xU>
+    <yV>-7.364</yV>
+    <zW>-17.955</zW>
+    <kP>-1.888</kP>
+    <mQ>-0.761</mQ>
+    <nR>-3.744</nR>
+    <!-- Negative quadratic damping -->
+    <xUU>-17.77</xUU>
+    <yVV>-125.9</yVV>
+    <zWW>-72.36</zWW>
+    <kPP>-0.1246</kPP>
+    <mQQ>-0.1246</mQQ>
+    <nRR>-0.1857</nRR>
     </plugin>
 </gazebo>

File: bluerov2_description/urdf/sensors.xacro (robot description, xacro)
@@ -9,17 +9,17 @@
             <mass value="0.015" />
         </inertial>
-      <xacro:if value="${simulation}">
+    </link>
+    <gazebo reference="${ns}/${name}">
         <sensor name="imu_sensor" type="imu">
             <always_on>1</always_on>
-            <update_rate>1</update_rate>
-            <visualize>true</visualize>
-            <topic>mpu</topic>
+            <update_rate>100</update_rate>
+            <visualize>false</visualize>
+            <topic>${ns}/${name}</topic>
         </sensor>
-        </xacro:if>
-    </link>
+    </gazebo>
      <joint name="${name}" type="fixed">
         <xacro:insert_block name="origin"/>
         <parent link="${ns}/base_link"/>
-        <child link="${ns}/${link_name}"/>
+        <child link="${ns}/${name}"/>
     </joint>
 </xacro:macro>
@@ -27,21 +27,9 @@
     <origin xyz="0 0 0" rpy="${PI} 0 0"/>
 </xacro:imu>
-  <!-- IMU Sensor -->
- <xacro:default_imu parent_link="${ns}/base_link" imu_name="mpu">
-    <origin xyz="0 0 0" rpy="${PI} 0 0"/>
-  </xacro:default_imu>
   <!-- Pressure Sensor  -->
-  <xacro:default_pressure parent_link="${ns}/base_link" sensor_name="baro">
+<!--  <xacro:default_pressure parent_link="${ns}/base_link" sensor_name="baro">
     <origin xyz="0 0 0" rpy="0 0 0"/>
-  </xacro:default_pressure>
- <!-- <link name="${ns}/camera">
-    <visual>
-    <geometry>
-        <cylinder radius="0.01" length="0.03"/>
-    </geometry>
-    <material name="black">
-        <color rgba="0 0 0 1"/>
-    </material>
-    </visual>
+  </xacro:default_pressure>-->
+  <link name="${ns}/camera">
     <inertial>
     <mass value="0.015"/>
@@ -54,10 +42,4 @@
     izz="0.001"/>
     </inertial>
-    <collision>
-      <geometry>
-        <cylinder length="${0.000001}" radius="${0.000001}" />
-      </geometry>
-      <origin xyz="0 0 0" rpy="0 ${0.5*pi} 0"/>
-    </collision>
  </link>
 <joint name="tilt" type="revolute">
@@ -66,40 +48,38 @@
     <origin xyz="${x_camera + .15} 0 0" rpy="0 ${PI/2} 0"/>
     <axis xyz="0 1 0" />
-    <limit effort="100" velocity="5.0" lower="${-PI/4}" upper="${PI/4}"/>
+    <limit effort="100" velocity="5.0" lower="${-PI/3}" upper="${PI/3}"/>
     <dynamics damping="0.8"/>
-</joint>-->
-<!--    <gazebo reference="${ns}/camera">
-        <material>Gazebo/Black</material>
+</joint>
+<gazebo>
+    <plugin filename="libignition-gazebo-joint-position-controller-system.so" name="ignition::gazebo::systems::JointPositionController">
+        <joint_name>tilt</joint_name>
+        <p_gain>1.</p_gain>
+        <i_gain>0.2</i_gain>
+        <d_gain>0.1</d_gain>
+        <i_max>10</i_max>
+        <i_min>-10</i_min>
+    </plugin>
+</gazebo>
+<xacro:if value="$(arg camera)">
+ <gazebo reference="${ns}/camera">
     <sensor name="camera" type="camera">
-      <update_rate>20</update_rate>
-      <camera name="camera">
-        <horizontal_fov>1.5125</horizontal_fov>
-        <image>
-          <width>768</width>
-          <height>492</height>
-          <format>R8G8B8</format>
-        </image>
-        <clip>
-          <near>0.2</near>
-          <far>200</far>
-        </clip>
-        <noise>
-          <type>gaussian</type>
-          <mean>0.0</mean>
-          <stddev>0.02</stddev>
-        </noise>
-      </camera>
-      <plugin filename="libgazebo_ros_camera.so" name="camera_controller">
-        <updateRate>20</updateRate>
-        <camera_name>${ns}/camera</camera_name>
-        <frame_name>${ns}/camera</frame_name>
-        <attenuationR>0.0</attenuationR>
-        <attenuationG>0.0</attenuationG>
-        <attenuationB>0.0</attenuationB>
-        <backgroundR>0</backgroundR>
-        <backgroundG>0</backgroundG>
-        <backgroundB>0</backgroundB>
-      </plugin>
-    </sensor>
-  </gazebo>-->
+    <camera>
+    <horizontal_fov>1.047</horizontal_fov> -->
+    <image>
+        <width>640</width>
+        <height>400</height>
+    </image>
+    <clip>
+        <near>0.3</near>
+        <far>100</far>
+    </clip>
+    </camera>
+    <always_on>1</always_on>
+    <update_rate>30</update_rate>
+    <visualize>true</visualize>
+    <topic>${ns}/image</topic>
+    <enable_metrics>false</enable_metrics>
+</sensor>
+  </gazebo>
+</xacro:if>
 </robot>

File: bluerov2_description/urdf/thrusters.xacro (robot description, xacro)
@@ -16,5 +16,5 @@
       <visual>
         <geometry>
-          <mesh filename="${prop_mesh_file}" scale="1 1 1" />
+          <mesh filename="${prop_mesh_file}"/>
         </geometry>
       </visual>
@@ -43,5 +43,5 @@
     </joint>
     <!-- ignition topic is /model/{ns}/joint/{joint_name}/cmd_thrust -->
-    <xacro:if value="$(arg simulation)">
+<!--     <xacro:if value="$(arg simulation)"> -->
     <gazebo>
         <plugin
@@ -51,13 +51,13 @@
             <joint_name>thruster${thruster_id}</joint_name>
 <!-- Thetys -->
+<!--            <thrust_coefficient>0.004422</thrust_coefficient>
+        <fluid_density>1000</fluid_density>
+        <propeller_diameter>0.2</propeller_diameter>-->
             <thrust_coefficient>0.004422</thrust_coefficient>
-        <fluid_density>1000</fluid_density>
-        <propeller_diameter>0.2</propeller_diameter>
-<!--            <thrust_coefficient>0.0001</thrust_coefficient>
             <fluid_density>${density}</fluid_density>
-            <propeller_diameter>${2*prop_r}</propeller_diameter>-->
+            <propeller_diameter>${2*prop_r}</propeller_diameter>
         </plugin>
     </gazebo>
-    </xacro:if>
+<!--     </xacro:if> -->
 </xacro:macro>
   <!-- all 6 thrusters -->

Commit message: scaled osg meshes, cascaded PID ok-ish

File: bluerov2_description/urdf/bluerov2.xacro (robot description, xacro)
@@ -12,10 +12,12 @@
   <xacro:property name="y_size" value="0.25"/>
   <xacro:property name="z_size" value="0.1"/>
-    <xacro:property name="mass" value="14.8"/>
+  <xacro:property name="mass" value="14.8"/>
   <!-- other props -->
   <xacro:property name="prop_mass" value="0.07"/>
   <xacro:property name="PI" value="3.1415927"/>
   <!-- to set correct buoyancy volume with 1 % positive factor -->
-  <xacro:property name="buoyant_correction" value="${pow(1.01*(mass + 6*prop_mass)/(density*x_size*y_size*z_size), 1./3)}"/>
+  <xacro:property name="buoyant_correction" value="${1.01*pow((mass + 6*prop_mass)/(density*x_size*y_size*z_size), 1./3)}"/>
+  <!-- Center of buoyancy -->
+  <xacro:property name="z_cob" value="${-buoyant_correction*z_size/4}"/>
   <!-- Center of gravity -->
   <xacro:property name="z_cog" value="${-buoyant_correction*z_size}"/>
@@ -44,4 +46,5 @@
     </visual>
     <collision>
+        <origin xyz="0 0 ${z_cob}"/>
         <!-- Box adjusted for buoyancy -->
         <geometry>
@@ -49,22 +52,29 @@
         </geometry>
     </collision>
+<!--    <gazebo>
+        <velocity_decay>
+            <linear>-250.15 -70.364 -170.955</linear>
+            <angular>1.888 0.761 3.744</angular>
+        </velocity_decay>
+</gazebo>-->
     </link>
 <xacro:include filename="hydrodynamics.xacro"/>
 <xacro:include filename="thrusters.xacro"/>
-  <xacro:include filename="sensors.xacro"/>
+<xacro:include filename="sensors.xacro"/>
 <!-- other Gazebo plugins -->
 <xacro:if value="$(arg simulation)">
     <gazebo>
-        <plugin filename="libignition-gazebo-joint-state-publisher-system.so" name="ignition::gazebo::systems::JointStatePublisher"/>
+        <plugin filename="gz-sim-joint-state-publisher-system" name="gz::sim::systems::JointStatePublisher"/>
         <plugin
-            filename="libignition-gazebo-odometry-publisher-system.so"
-            name="ignition::gazebo::systems::OdometryPublisher">
+            filename="gz-sim-odometry-publisher-system"
+            name="gz::sim::systems::OdometryPublisher">
             <odom_frame>${ns}/odom</odom_frame>
+            <dimensions>3</dimensions>
             <robot_base_frame>${ns}/base_link</robot_base_frame>
             <odom_publish_frequency>10</odom_publish_frequency>
         </plugin>
         <plugin
-            filename="libignition-gazebo-pose-publisher-system.so"
-            name="ignition::gazebo::systems::PosePublisher">
+            filename="gz-sim-pose-publisher-system"
+            name="gz::sim::systems::PosePublisher">
             <publish_link_pose>false</publish_link_pose>
             <publish_collision_pose>false</publish_collision_pose>

File: bluerov2_description/urdf/hydrodynamics.xacro (robot description, xacro)
@@ -1,19 +1,24 @@
 <?xml version="1.0"?>
-<robot xmlns:xacro="http://www.ros.org/wiki/xacro">
+<xacro>
 <gazebo>
-    <plugin
-filename="libignition-gazebo-hydrodynamics-system.so"
-name="ignition::gazebo::systems::Hydrodynamics">
+    <plugin filename="gz-sim-hydrodynamics-system" name="gz::sim::systems::Hydrodynamics">
+<!--     <density>${density}</density> -->
     <!-- Ignition notations from Handbook of Marine Craft, Fossen, 2011 -->
     <link_name>${ns}/base_link</link_name>
+     <xU>0</xU>
+      <yV>0</yV>
+      <zW>0</zW>
+      <kP>0</kP>
+      <mQ>0</mQ>
+      <nR>0</nR>
     <!-- BlueROV2 heavy values from "6-DoF Modelling and Control of a Remotely Operated Vehicle"
         Wu, Master thesis, Flinder University, 2018  -->
     <!-- Negative diagonal values of added mass matrix [Fossen (6.38)] -->
-    <xDotU>-5.5</xDotU>
+<!--    <xDotU>-5.5</xDotU>
     <yDotV>-12.7</yDotV>
     <zDotW>-14.57</zDotW>
     <kDotP>-0.12</kDotP>
     <mDotQ>-0.12</mDotQ>
-    <nDotR>-0.12</nDotR>
+    <nDotR>-0.12</nDotR>-->
     <!-- From "Numerical Modelling and Experimental Testing of the Hydrodynamic Characteristics
         for an Open-Frame Remotely Operated Vehicle",  Li et al, Marine Science and Engineering, 2020         -->
@@ -26,27 +31,27 @@
     <nR>-0.</nR>-->
     <!-- Negative quadratic damping [Fossen (6.62)] -->
-<!--    <xUU>38.169</xUU>
-    <yVV>-129.66</yVV>
-    <zWW>-243.25</zWW>
-    <kPP>-4.86</kPP>
-    <mQQ>-4.86</mQQ>
-    <nRR>-4.86</nRR>-->
+      <xUabsU>-33.800000000000004</xUabsU>
+      <yVabsV>-54.26875</yVabsV>
+      <zWabsW>-73.37135</zWabsW>
+      <kPabsP>-4.0</kPabsP>
+      <mQabsQ>-4.0</mQabsQ>
+      <nRabsR>-4.0</nRabsR>
     <!-- BlueROV2 values from "Model Predictive Control for the BlueROV2",
         Emil Már Einarsson, Andris Lipenitis, Master thesis, 2020  -->
     <!-- Negative linear damping -->
-    <xU>-25.15</xU>
+<!--    <xU>-25.15</xU>
     <yV>-7.364</yV>
     <zW>-17.955</zW>
     <kP>-1.888</kP>
     <mQ>-0.761</mQ>
-    <nR>-3.744</nR>
+    <nR>-3.744</nR>-->
     <!-- Negative quadratic damping -->
-    <xUU>-17.77</xUU>
+<!--    <xUU>-17.77</xUU>
     <yVV>-125.9</yVV>
     <zWW>-72.36</zWW>
     <kPP>-0.1246</kPP>
     <mQQ>-0.1246</mQQ>
-    <nRR>-0.1857</nRR>
+    <nRR>-0.1857</nRR>-->
     </plugin>
 </gazebo>
-</robot>
+</xacro>

File: bluerov2_description/urdf/sensors.xacro (robot description, xacro)
@@ -9,12 +9,17 @@
             <mass value="0.015" />
         </inertial>
+        <sensor name="${name}_imu" type="imu">
+            <always_on>1</always_on>
+            <update_rate>1</update_rate>
+            <visualize>true</visualize>
+            <topic>${name}</topic>
+        </sensor>
     </link>
     <gazebo reference="${ns}/${name}">
-        <sensor name="imu_sensor" type="imu">
-            <always_on>1</always_on>
-            <update_rate>100</update_rate>
-            <visualize>false</visualize>
-            <topic>${ns}/${name}</topic>
-        </sensor>
+         <plugin
+            filename="libgz-sim-imu-system.so"
+            name="gz::sim::systems::Imu">
+             <link_name>${ns}/${name}</link_name>
+        </plugin>
     </gazebo>
      <joint name="${name}" type="fixed">
@@ -25,5 +30,8 @@
 </xacro:macro>
 <xacro:imu name="mpu">
-    <origin xyz="0 0 0" rpy="${PI} 0 0"/>
+    <origin xyz="0.1 0 0" rpy="0 0 ${-PI/2}"/>
+</xacro:imu>
+<xacro:imu name="lsm">
+    <origin xyz="0.1 0 0" rpy="0 0 ${-PI/2}"/>
 </xacro:imu>
   <!-- Pressure Sensor  -->
@@ -52,5 +60,5 @@
 </joint>
 <gazebo>
-    <plugin filename="libignition-gazebo-joint-position-controller-system.so" name="ignition::gazebo::systems::JointPositionController">
+    <plugin filename="gz-sim-joint-position-controller-system" name="gz::sim::systems::JointPositionController">
         <joint_name>tilt</joint_name>
         <topic>${ns}/tilt_cmd</topic>

File: bluerov2_description/urdf/thrusters.xacro (robot description, xacro)
@@ -2,5 +2,5 @@
 <robot xmlns:xacro="http://www.ros.org/wiki/xacro">
   <xacro:property name="prop_mesh_file" value="file://$(find bluerov2_description)/meshes/bluerov2_propcw.dae"/>
-  <xacro:property name="prop_r" value="0.038"/>
+  <xacro:property name="prop_r" value="0.05"/>
   <xacro:property name="prop_l" value="0.035"/>
   <!--  Thruster macro: joint + link + plugin -->
@@ -12,10 +12,10 @@
         </geometry>
       </visual>
-        <collision>
+<!--        <collision>
             <origin rpy="0 ${PI/2} 0"/>
         <geometry>
             <cylinder length="${prop_l}" radius="${prop_r}"/>
         </geometry>
-      </collision>
+      </collision>-->
      <inertial>
      <!-- thruster axis is X -->
@@ -39,11 +39,14 @@
     <gazebo>
         <plugin
-            filename="ignition-gazebo-thruster-system"
-            name="ignition::gazebo::systems::Thruster">
+            filename="gz-sim-thruster-system"
+            name="gz::sim::systems::Thruster">
             <namespace>${ns}</namespace>
             <joint_name>thruster${thruster_id}</joint_name>
-            <thrust_coefficient>0.004422</thrust_coefficient>
+            <topic>thruster${thruster_id}/cmd</topic>
+            <thrust_coefficient>0.02</thrust_coefficient>
             <fluid_density>${density}</fluid_density>
             <propeller_diameter>${2*prop_r}</propeller_diameter>
+            <velocity_control>true</velocity_control>
+            <use_angvel_cmd>false</use_angvel_cmd>
         </plugin>
     </gazebo>
