Commit message: back to ignition ns to test on Foxy

File: bluerov2_description/urdf/bluerov2.xacro (robot description, xacro)
@@ -14,5 +14,4 @@
   <!-- other props -->
   <xacro:property name="prop_mass" value="0.07"/>
-  <xacro:property name="PI" value="3.1415927"/>
   <!-- to set correct buoyancy volume with 1 % positive factor -->
   <xacro:property name="buoyant_correction" value="${1.01*pow((mass + 6*prop_mass)/(density*x_size*y_size*z_size), 1./3)}"/>
@@ -64,8 +63,8 @@
 <xacro:if value="$(arg simulation)">
     <gazebo>
-        <plugin filename="gz-sim-joint-state-publisher-system" name="gz::sim::systems::JointStatePublisher"/>
+        <plugin filename="gz-sim-joint-state-publisher-system" name="ignition::gazebo::systems::JointStatePublisher"/>
         <plugin
-            filename="gz-sim-odometry-publisher-system"
-            name="gz::sim::systems::OdometryPublisher">
+            filename="ignition-gazebo-odometry-publisher-system"
+            name="ignition::gazebo::systems::OdometryPublisher">
             <odom_frame>${ns}/odom</odom_frame>
             <dimensions>3</dimensions>
@@ -74,6 +73,6 @@
         </plugin>
         <plugin
-            filename="gz-sim-pose-publisher-system"
-            name="gz::sim::systems::PosePublisher">
+            filename="ignition-gazebo-pose-publisher-system"
+            name="ignition::gazebo::systems::PosePublisher">
             <publish_link_pose>false</publish_link_pose>
             <publish_collision_pose>false</publish_collision_pose>

File: bluerov2_description/urdf/hydrodynamics.xacro (robot description, xacro)
@@ -2,5 +2,5 @@
 <xacro>
 <gazebo>
-    <plugin filename="gz-sim-hydrodynamics-system" name="gz::sim::systems::Hydrodynamics">
+    <plugin filename="gz-sim-hydrodynamics-system" name="ignition::gazebo::systems::Hydrodynamics">
 <!--     <density>${density}</density> -->
     <!-- Ignition notations from Handbook of Marine Craft, Fossen, 2011 -->

File: bluerov2_description/urdf/sensors.xacro (robot description, xacro)
@@ -181,5 +181,5 @@
 </gazebo>
 <gazebo>
-    <plugin filename="gz-sim-joint-position-controller-system" name="gz::sim::systems::JointPositionController">
+    <plugin filename="gz-sim-joint-position-controller-system" name="ignition::gazebo::systems::JointPositionController">
         <joint_name>tilt</joint_name>
         <p_gain>10.</p_gain>

File: bluerov2_description/urdf/thrusters.xacro (robot description, xacro)
@@ -1,5 +1,6 @@
 <?xml version="1.0"?>
 <robot xmlns:xacro="http://www.ros.org/wiki/xacro">
-  <xacro:property name="prop_mesh_file" value="file://$(find bluerov2_description)/meshes/bluerov2_propcw.dae"/>
+  <xacro:property name="prop_mesh_cw" value="file://$(find bluerov2_description)/meshes/bluerov2_propcw.dae"/>
+  <xacro:property name="prop_mesh_ccw" value="file://$(find bluerov2_description)/meshes/bluerov2_propccw.dae"/>
   <xacro:property name="prop_r" value="0.05"/>
   <xacro:property name="prop_l" value="0.035"/>
@@ -9,5 +10,10 @@
       <visual>
         <geometry>
-          <mesh filename="${prop_mesh_file}"/>
+          <xacro:if value="${thruster_id in [1,2,5]}">
+            <mesh filename="${prop_mesh_cw}"/>
+          </xacro:if>
+            <xacro:unless value="${thruster_id in [1,2,5]}">
+            <mesh filename="${prop_mesh_ccw}"/>
+          </xacro:unless>
         </geometry>
       </visual>
@@ -30,5 +36,10 @@
     <joint name="thruster${thruster_id}" type="continuous">
       <xacro:insert_block name="origin" />
-      <axis xyz="1 0 0" />
+      <xacro:if value="${thruster_id in [1,2,5]}">
+        <axis xyz="1 0 0" />
+      </xacro:if>
+      <xacro:unless value="${thruster_id in [1,2,5]}">
+        <axis xyz="-1 0 0" />
+      </xacro:unless>
       <parent link="${ns}/base_link" />
       <child link="${ns}/thruster${thruster_id}" />
@@ -39,6 +50,6 @@
     <gazebo>
         <plugin
-            filename="gz-sim-thruster-system"
-            name="gz::sim::systems::Thruster">
+            filename="ignition-gazebo-thruster-system"
+            name="ignition::gazebo::systems::Thruster">
             <namespace>${ns}</namespace>
             <joint_name>thruster${thruster_id}</joint_name>

Commit message: use package:// meshes with Gazebo env hooks

File: bluerov2_description/urdf/bluerov2.xacro (robot description, xacro)
@@ -20,6 +20,6 @@
   <!-- Center of gravity -->
   <xacro:property name="z_cog" value="${-buoyant_correction*z_size}"/>
-  <xacro:property name="visual_mesh_file" value="file://$(find bluerov2_description)/meshes/bluerov2_noprop.dae"/>
-  <xacro:property name="collision_mesh_file" value="file://$(find bluerov2_description)/meshes/bluerov2_noprop.stl"/>
+  <xacro:property name="visual_mesh_file" value="package://bluerov2_description/meshes/bluerov2_noprop.dae"/>
+  <xacro:property name="collision_mesh_file" value="package://bluerov2_description/meshes/bluerov2_noprop.stl"/>
   <!-- Vehicle base link -->
     <link name="${ns}/base_link">

File: bluerov2_description/urdf/sensors.xacro (robot description, xacro)
@@ -8,9 +8,8 @@
     <sensor name="${name}_imu" type="imu">
             <always_on>1</always_on>
-            <update_rate>1</update_rate>
+            <update_rate>10</update_rate>
             <visualize>true</visualize>
             <topic>${ns}/${name}</topic>
             <gz_frame_id>${ns}/${name}</gz_frame_id>
-            <update_rate>100</update_rate>
       <imu>
         <angular_velocity>
@@ -136,5 +135,5 @@
       <origin xyz="0 0 -0.022" rpy="0 0 0"/>
       <geometry>
-        <mesh filename="file://$(find bluerov2_description)/meshes/ping360_sonar.dae"
+        <mesh filename="package://bluerov2_description/meshes/ping360_sonar.dae"
               scale="0.01 0.01 0.01"/>/>
       </geometry>

File: bluerov2_description/urdf/thrusters.xacro (robot description, xacro)
@@ -1,6 +1,6 @@
 <?xml version="1.0"?>
 <robot xmlns:xacro="http://www.ros.org/wiki/xacro">
-  <xacro:property name="prop_mesh_cw" value="file://$(find bluerov2_description)/meshes/bluerov2_propcw.dae"/>
-  <xacro:property name="prop_mesh_ccw" value="file://$(find bluerov2_description)/meshes/bluerov2_propccw.dae"/>
+  <xacro:property name="prop_mesh_cw" value="package://bluerov2_description/meshes/bluerov2_propcw.dae"/>
+  <xacro:property name="prop_mesh_ccw" value="package://bluerov2_description/meshes/bluerov2_propccw.dae"/>
   <xacro:property name="prop_r" value="0.05"/>
   <xacro:property name="prop_l" value="0.035"/>
