Commit message: gz::sim plugins

File: bluerov2_description/urdf/bluerov2.xacro (robot description, xacro)
@@ -63,8 +63,8 @@
 <xacro:if value="$(arg simulation)">
     <gazebo>
-        <plugin filename="ignition-gazebo-joint-state-publisher-system" name="ignition::gazebo::systems::JointStatePublisher"/>
+        <plugin filename="gz-sim-joint-state-publisher-system" name="gz::sim::systems::JointStatePublisher"/>
         <plugin
-            filename="ignition-gazebo-odometry-publisher-system"
-            name="ignition::gazebo::systems::OdometryPublisher">
+            filename="gz-sim-odometry-publisher-system"
+            name="gz::sim::systems::OdometryPublisher">
             <odom_frame>world</odom_frame>
             <dimensions>3</dimensions>
@@ -73,6 +73,6 @@
         </plugin>
         <plugin
-            filename="ignition-gazebo-pose-publisher-system"
-            name="ignition::gazebo::systems::PosePublisher">
+            filename="gz-sim-pose-publisher-system"
+            name="gz::sim::systems::PosePublisher">
             <publish_link_pose>false</publish_link_pose>
             <publish_collision_pose>false</publish_collision_pose>

File: bluerov2_description/urdf/hydrodynamics.xacro (robot description, xacro)
@@ -2,5 +2,5 @@
 <xacro>
 <gazebo>
-    <plugin filename="ignition-gazebo-hydrodynamics-system" name="ignition::gazebo::systems::Hydrodynamics">
+    <plugin filename="gz-sim-hydrodynamics-system" name="gz::sim::systems::Hydrodynamics">
 <!--     <density>${density}</density> -->
     <!-- Ignition notations from Handbook of Marine Craft, Fossen, 2011 -->

File: bluerov2_description/urdf/sensors.xacro (robot description, xacro)
@@ -101,5 +101,5 @@
 </xacro:imu>-->
 <xacro:imu name="imu">
-    <origin xyz="0.058 -0.021 0.018" rpy="${pi/2} 0 0"/>
+    <origin xyz="0.058 -0.021 0.018" rpy="0 0 0"/> <!--${pi/2}-->
 </xacro:imu>
   <!-- Pressure Sensor  -->
@@ -182,5 +182,5 @@
 </gazebo>
 <gazebo>
-    <plugin filename="ignition-gazebo-joint-position-controller-system" name="ignition::gazebo::systems::JointPositionController">
+    <plugin filename="gz-sim-joint-position-controller-system" name="gz::sim::systems::JointPositionController">
         <joint_name>tilt</joint_name>
         <p_gain>10.</p_gain>

File: bluerov2_description/urdf/thrusters.xacro (robot description, xacro)
@@ -50,6 +50,6 @@
     <gazebo>
         <plugin
-            filename="ignition-gazebo-thruster-system"
-            name="ignition::gazebo::systems::Thruster">
+            filename="gz-sim-thruster-system"
+            name="gz::sim::systems::Thruster">
             <namespace>${ns}</namespace>
             <joint_name>thruster${thruster_id}</joint_name>
@@ -68,14 +68,14 @@
   <!-- all 6 thrusters -->
   <xacro:thruster thruster_id="1">
-    <origin xyz="0.1355 -0.1 -0.0725" rpy="0 0 0.7853981634"/>
+    <origin xyz="0.1355 -0.1 -0.0725" rpy="0 0 -2.3561944902"/>
   </xacro:thruster>
   <xacro:thruster thruster_id="2">
-    <origin xyz="0.1355 0.1 -0.0725" rpy="0 0 -0.7853981634"/>
+    <origin xyz="0.1355 0.1 -0.0725" rpy="0 0 2.3561944902"/>
   </xacro:thruster>
   <xacro:thruster thruster_id="3">
-    <origin xyz="-0.1475 -0.1 -0.0725" rpy="0 0 2.3561944902"/>
+    <origin xyz="-0.1475 -0.1 -0.0725" rpy="0 0 -0.7853981634"/>
   </xacro:thruster>
   <xacro:thruster thruster_id="4">
-    <origin xyz="-0.1475 0.1 -0.0725" rpy="0 0 -2.3561944902"/>
+    <origin xyz="-0.1475 0.1 -0.0725" rpy="0 0 0.7853981634"/>
   </xacro:thruster>
   <xacro:thruster thruster_id="5">
