Commit message: remove use_sim_time from config file

File: bluerov2_description/urdf/sensors.xacro (robot description, xacro)
@@ -54,4 +54,5 @@
     <plugin filename="libignition-gazebo-joint-position-controller-system.so" name="ignition::gazebo::systems::JointPositionController">
         <joint_name>tilt</joint_name>
+        <topic>${ns}/tilt_cmd</topic>
         <p_gain>1.</p_gain>
         <i_gain>0.2</i_gain>
@@ -65,5 +66,5 @@
     <sensor name="camera" type="camera">
     <camera>
-    <horizontal_fov>1.047</horizontal_fov> -->
+    <horizontal_fov>1.047</horizontal_fov>
     <image>
         <width>640</width>

File: bluerov2_description/urdf/thrusters.xacro (robot description, xacro)
@@ -4,11 +4,4 @@
   <xacro:property name="prop_r" value="0.038"/>
   <xacro:property name="prop_l" value="0.035"/>
-  <xacro:if value="$(arg simulation)">
-    <!-- Gazebo needs thrusters to rotate -->
-    <xacro:property name="thruster_joint_type" value="continuous"/>
-  </xacro:if>
-  <xacro:unless value="$(arg simulation)">
-      <xacro:property name="thruster_joint_type" value="fixed"/>
-  </xacro:unless>
   <!--  Thruster macro: joint + link + plugin -->
   <xacro:macro name="thruster" params="thruster_id *origin">
@@ -35,5 +28,5 @@
     </link>
     <!-- Joint between thruster link and vehicle base link -->
-    <joint name="thruster${thruster_id}" type="${thruster_joint_type}">
+    <joint name="thruster${thruster_id}" type="continuous">
       <xacro:insert_block name="origin" />
       <axis xyz="1 0 0" />
@@ -42,6 +35,6 @@
       <limits effort="-1" velocity="-1"/>
     </joint>
-    <!-- ignition topic is /model/{ns}/joint/{joint_name}/cmd_thrust -->
-<!--     <xacro:if value="$(arg simulation)"> -->
+    <!-- ignition topic is /model/{ns}/joint/{joint_name}/cmd_pos -->
+<!--    <xacro:if value="$(arg simulation)"> -->
     <gazebo>
         <plugin
@@ -50,8 +43,4 @@
             <namespace>${ns}</namespace>
             <joint_name>thruster${thruster_id}</joint_name>
-<!-- Thetys -->
-<!--            <thrust_coefficient>0.004422</thrust_coefficient>
-        <fluid_density>1000</fluid_density>
-        <propeller_diameter>0.2</propeller_diameter>-->
             <thrust_coefficient>0.004422</thrust_coefficient>
             <fluid_density>${density}</fluid_density>
@@ -59,5 +48,5 @@
         </plugin>
     </gazebo>
-<!--     </xacro:if> -->
+<!--  </xacro:if> -->
 </xacro:macro>
   <!-- all 6 thrusters -->

Commit message: move tilt config to control package

File: bluerov2_description/urdf/sensors.xacro (robot description, xacro)
@@ -54,8 +54,14 @@
     <parent link="${ns}/base_link"/>
     <child link="${ns}/camera"/>
-    <origin xyz="${x_camera + .15} 0 0" rpy="0 ${PI/2} 0"/>
+    <origin xyz="${x_camera + .15} 0 0" rpy="0 0 0"/>
     <axis xyz="0 1 0" />
     <limit effort="100" velocity="5.0" lower="${-PI/3}" upper="${PI/3}"/>
     <dynamics damping="0.8"/>
+</joint>
+<link name="${ns}/camera_optical"/>
+<joint name="camera_optical" type="fixed">
+    <parent link="${ns}/camera"/>
+    <child link="${ns}/camera_optical"/>
+    <origin rpy="${-PI/2} 0 ${-PI/2}"/>
 </joint>
 <gazebo>

Commit message: custom underwater world with buoyancy + thrusters

File: bluerov2_description/urdf/sensors.xacro (robot description, xacro)
@@ -5,22 +5,88 @@
 <xacro:macro name="imu" params="name *origin">
     <link name="${ns}/${name}">
-        <inertial>
-            <inertia ixx="0.00001" ixy="0.0" ixz="0.0" iyy="0.00001" iyz="0.0" izz="0.00001" />
-            <mass value="0.015" />
-        </inertial>
         <sensor name="${name}_imu" type="imu">
             <always_on>1</always_on>
             <update_rate>1</update_rate>
             <visualize>true</visualize>
-            <topic>${name}</topic>
+            <topic>${ns}/${name}</topic>
+            <gz_frame_id>${ns}/${name}</gz_frame_id>
+            <update_rate>100</update_rate>
+      <imu>
+        <angular_velocity>
+          <x>
+            <noise type="gaussian">
+              <mean>0</mean>
+              <stddev>0.009</stddev>
+              <bias_mean>0.00075</bias_mean>
+              <bias_stddev>0.005</bias_stddev>
+              <dynamic_bias_stddev>0.00002</dynamic_bias_stddev>
+              <dynamic_bias_correlation_time>400.0</dynamic_bias_correlation_time>
+              <precision>0.00025</precision>
+            </noise>
+          </x>
+          <y>
+            <noise type="gaussian">
+              <mean>0</mean>
+              <stddev>0.009</stddev>
+              <bias_mean>0.00075</bias_mean>
+              <bias_stddev>0.005</bias_stddev>
+              <dynamic_bias_stddev>0.00002</dynamic_bias_stddev>
+              <dynamic_bias_correlation_time>400.0</dynamic_bias_correlation_time>
+              <precision>0.00025</precision>
+            </noise>
+          </y>
+          <z>
+            <noise type="gaussian">
+              <mean>0</mean>
+              <stddev>0.009</stddev>
+              <bias_mean>0.00075</bias_mean>
+              <bias_stddev>0.005</bias_stddev>
+              <dynamic_bias_stddev>0.00002</dynamic_bias_stddev>
+              <dynamic_bias_correlation_time>400.0</dynamic_bias_correlation_time>
+              <precision>0.00025</precision>
+            </noise>
+          </z>
+        </angular_velocity>
+        <linear_acceleration>
+          <x>
+            <noise type="gaussian">
+              <mean>0</mean>
+              <stddev>0.021</stddev>
+              <bias_mean>0.05</bias_mean>
+              <bias_stddev>0.0075</bias_stddev>
+              <dynamic_bias_stddev>0.000375</dynamic_bias_stddev>
+              <dynamic_bias_correlation_time>175.0</dynamic_bias_correlation_time>
+              <precision>0.005</precision>
+            </noise>
+          </x>
+          <y>
+            <noise type="gaussian">
+              <mean>0</mean>
+              <stddev>0.021</stddev>
+              <bias_mean>0.05</bias_mean>
+              <bias_stddev>0.0075</bias_stddev>
+              <dynamic_bias_stddev>0.000375</dynamic_bias_stddev>
+              <dynamic_bias_correlation_time>175.0</dynamic_bias_correlation_time>
+              <precision>0.005</precision>
+            </noise>
+          </y>
+          <z>
+            <noise type="gaussian">
+              <mean>0</mean>
+              <stddev>0.021</stddev>
+              <bias_mean>0.05</bias_mean>
+              <bias_stddev>0.0075</bias_stddev>
+              <dynamic_bias_stddev>0.000375</dynamic_bias_stddev>
+              <dynamic_bias_correlation_time>175.0</dynamic_bias_correlation_time>
+              <precision>0.005</precision>
+            </noise>
+          </z>
+        </linear_acceleration>
+        <orientation_reference_frame>
+          <localization>ENU</localization>
+        </orientation_reference_frame>
+      </imu>
         </sensor>
     </link>
-    <gazebo reference="${ns}/${name}">
-         <plugin
-            filename="libgz-sim-imu-system.so"
-            name="gz::sim::systems::Imu">
-             <link_name>${ns}/${name}</link_name>
-        </plugin>
-    </gazebo>
      <joint name="${name}" type="fixed">
         <xacro:insert_block name="origin"/>

File: bluerov2_description/urdf/thrusters.xacro (robot description, xacro)
@@ -50,5 +50,5 @@
             <use_angvel_cmd>false</use_angvel_cmd>
         </plugin>
-    </gazebo>
+      </gazebo>
 <!--  </xacro:if> -->
 </xacro:macro>

Commit message: add IMU simulation

File: bluerov2_description/urdf/sensors.xacro (robot description, xacro)
@@ -4,6 +4,7 @@
 <xacro:property name="PI" value="3.1415927"/>
 <xacro:macro name="imu" params="name *origin">
-    <link name="${ns}/${name}">
-        <sensor name="${name}_imu" type="imu">
+    <link name="${ns}/${name}"/>
+    <gazebo reference="${ns}/${name}">
+    <sensor name="${name}_imu" type="imu">
             <always_on>1</always_on>
             <update_rate>1</update_rate>
@@ -88,5 +89,5 @@
       </imu>
         </sensor>
-    </link>
+      </gazebo>
      <joint name="${name}" type="fixed">
         <xacro:insert_block name="origin"/>

Commit message: add ping360 sonar, simulated as laserscan for now

File: bluerov2_description/urdf/sensors.xacro (robot description, xacro)
@@ -132,4 +132,46 @@
     <origin rpy="${-PI/2} 0 ${-PI/2}"/>
 </joint>
+<link name="${ns}/sonar">
+    <visual>
+      <origin xyz="0 0 -0.022" rpy="0 0 ${PI/2}"/>
+      <geometry>
+        <mesh filename="file://$(find bluerov2_description)/meshes/ping360_sonar.dae"
+              scale="0.01 0.01 0.01"/>/>
+      </geometry>
+    </visual>
+</link>
+<joint name="sonar" type="fixed">
+    <parent link="${ns}/base_link"/>
+    <child link="${ns}/sonar"/>
+    <origin xyz="0.135 0.108 0.118"/>
+</joint>
+<gazebo reference="${ns}/sonar">
+  <sensor type="gpu_lidar" name="ping360_sonar">
+    <pose>0 0 0 0 0 0</pose>
+    <update_rate>5</update_rate>
+    <topic>${ns}/sonar</topic>
+    <gz_frame_id>${ns}/sonar</gz_frame_id>
+    <ray>
+      <scan>
+        <horizontal>
+          <samples>360</samples>
+          <resolution>1</resolution>
+          <min_angle>0.0</min_angle>
+          <max_angle>6.28319</max_angle>
+        </horizontal>
+      </scan>
+      <range>
+        <min>0.1</min>
+        <max>20.</max>
+        <resolution>0.015</resolution>
+      </range>
+      <noise>
+        <type>gaussian</type>
+        <mean>0.0</mean>
+        <stddev>0.01</stddev>
+      </noise>
+    </ray>
+  </sensor>
+</gazebo>
 <gazebo>
     <plugin filename="gz-sim-joint-position-controller-system" name="gz::sim::systems::JointPositionController">
@@ -143,5 +185,5 @@
 </gazebo>
  <gazebo reference="${ns}/camera">
-    <sensor name="camera" type="camera">
+  <sensor name="camera" type="camera">
     <camera>
     <optical_frame_id>${ns}/camera_optical</optical_frame_id>

Commit message: Z-up in sonar

File: bluerov2_description/urdf/sensors.xacro (robot description, xacro)
@@ -134,5 +134,5 @@
 <link name="${ns}/sonar">
     <visual>
-      <origin xyz="0 0 -0.022" rpy="0 0 ${PI/2}"/>
+      <origin xyz="0 0 -0.022" rpy="0 0 0"/>
       <geometry>
         <mesh filename="file://$(find bluerov2_description)/meshes/ping360_sonar.dae"

Commit message: add imu frame for real one

File: bluerov2_description/urdf/sensors.xacro (robot description, xacro)
@@ -98,5 +98,8 @@
     <origin xyz="0.1 0 0" rpy="0 0 ${-PI/2}"/>
 </xacro:imu>
-<xacro:imu name="lsm">
+<xacro:imu name="mpu">
+    <origin xyz="0.1 0 0" rpy="0 0 ${-PI/2}"/>
+</xacro:imu>
+<xacro:imu name="imu">
     <origin xyz="0.1 0 0" rpy="0 0 ${-PI/2}"/>
 </xacro:imu>

Commit message: sonar

File: bluerov2_description/urdf/sensors.xacro (robot description, xacro)
@@ -146,5 +146,5 @@
     <parent link="${ns}/base_link"/>
     <child link="${ns}/sonar"/>
-    <origin xyz="0.135 0.108 0.118"/>
+    <origin xyz="0.135 -0.108 0.118"/>
 </joint>
 <gazebo reference="${ns}/sonar">

Commit message: correct ? imu placement

File: bluerov2_description/urdf/sensors.xacro (robot description, xacro)
@@ -2,5 +2,4 @@
 <robot xmlns:xacro="http://www.ros.org/wiki/xacro">
 <xacro:property name="x_camera" value="0.02"/>
-<xacro:property name="PI" value="3.1415927"/>
 <xacro:macro name="imu" params="name *origin">
     <link name="${ns}/${name}"/>
@@ -96,11 +95,11 @@
 </xacro:macro>
 <xacro:imu name="mpu">
-    <origin xyz="0.1 0 0" rpy="0 0 ${-PI/2}"/>
+    <origin xyz="0.1 0 0" rpy="0 0 ${-pi/2}"/>
 </xacro:imu>
-<xacro:imu name="mpu">
-    <origin xyz="0.1 0 0" rpy="0 0 ${-PI/2}"/>
+<xacro:imu name="lsm">
+    <origin xyz="0.1 0 0" rpy="0 0 ${-pi/2}"/>
 </xacro:imu>
 <xacro:imu name="imu">
-    <origin xyz="0.1 0 0" rpy="0 0 ${-PI/2}"/>
+    <origin xyz="0.058 -0.021 0.018" rpy="${pi/2} 0 0"/>
 </xacro:imu>
   <!-- Pressure Sensor  -->
@@ -125,5 +124,5 @@
     <origin xyz="${x_camera + .15} 0 0" rpy="0 0 0"/>
     <axis xyz="0 1 0" />
-    <limit effort="100" velocity="5.0" lower="${-PI/3}" upper="${PI/3}"/>
+    <limit effort="100" velocity="5.0" lower="${-pi/3}" upper="${pi/3}"/>
     <dynamics damping="0.8"/>
 </joint>
@@ -132,5 +131,5 @@
     <parent link="${ns}/camera"/>
     <child link="${ns}/camera_optical"/>
-    <origin rpy="${-PI/2} 0 ${-PI/2}"/>
+    <origin rpy="${-pi/2} 0 ${-pi/2}"/>
 </joint>
 <link name="${ns}/sonar">
